Commit message: Fixed description download files

File: catkin_ws/src/gen2_description/urdf/gen2.xacro (robot description, xacro)
@@ -1,1156 +1,550 @@
-<!DOCTYPE html>
-<html>
-  <head prefix="og: http://ogp.me/ns# fb: http://ogp.me/ns/fb# githubog: http://ogp.me/ns/fb/githubog#">
-    <meta charset='utf-8'>
-    <meta http-equiv="X-UA-Compatible" content="IE=edge">
-        <title>Gen2_Platforms_old/gen2_common/gen2_description/urdf/gen2.xacro at master · crrlab368/Gen2_Platforms_old</title>
-    <link rel="search" type="application/opensearchdescription+xml" href="/opensearch.xml" title="GitHub" />
-    <link rel="fluid-icon" href="https://github.com/fluidicon.png" title="GitHub" />
-    <link rel="apple-touch-icon" sizes="57x57" href="/apple-touch-icon-114.png" />
-    <link rel="apple-touch-icon" sizes="114x114" href="/apple-touch-icon-114.png" />
-    <link rel="apple-touch-icon" sizes="72x72" href="/apple-touch-icon-144.png" />
-    <link rel="apple-touch-icon" sizes="144x144" href="/apple-touch-icon-144.png" />
-    <link rel="logo" type="image/svg" href="http://github-media-downloads.s3.amazonaws.com/github-logo.svg" />
-    <link rel="xhr-socket" href="/_sockets" />
-    <meta name="msapplication-TileImage" content="/windows-tile.png" />
-    <meta name="msapplication-TileColor" content="#ffffff" />
-    <meta name="selected-link" value="repo_source" data-pjax-transient />
-    <meta content="collector.githubapp.com" name="octolytics-host" /><meta content="github" name="octolytics-app-id" /><meta content="954816" name="octolytics-actor-id" /><meta content="332534291b9b200342d8b1864dfd3db081ffed2411bc4e63e6334b139e1e54e0" name="octolytics-actor-hash" />
-    <link rel="icon" type="image/x-icon" href="/favicon.ico" />
-    <meta content="authenticity_token" name="csrf-param" />
-<meta content="vWZ31DoCO0bdiK1SaFbgMAphXvwWP/Ea7z/IJlIrUBA=" name="csrf-token" />
-    <link href="https://a248.e.akamai.net/assets.github.com/assets/github-159290696eb4150b6abdc4ac7fa8da500bcca10f.css" media="all" rel="stylesheet" type="text/css" />
-    <link href="https://a248.e.akamai.net/assets.github.com/assets/github2-2c49c2224329e588ccb1cf3d6450086dc1cff047.css" media="all" rel="stylesheet" type="text/css" />
-      <script src="https://a248.e.akamai.net/assets.github.com/assets/frameworks-92d138f450f2960501e28397a2f63b0f100590f0.js" type="text/javascript"></script>
-      <script src="https://a248.e.akamai.net/assets.github.com/assets/github-76cc892ab78e865420ada4b851fbb109aa83cbfc.js" type="text/javascript"></script>
-      <meta http-equiv="x-pjax-version" content="d35cab367dbc001c05b2c7abe21106cb">
-        <link data-pjax-transient rel='permalink' href='/crrlab368/Gen2_Platforms_old/blob/5cf94742cfdbf212b6ec9cc24dc8148d8ee83f12/gen2_common/gen2_description/urdf/gen2.xacro'>
-    <meta property="og:title" content="Gen2_Platforms_old"/>
-    <meta property="og:type" content="githubog:gitrepository"/>
-    <meta property="og:url" content="https://github.com/crrlab368/Gen2_Platforms_old"/>
-    <meta property="og:image" content="https://secure.gravatar.com/avatar/9f67947d0c852e39e3bd1cf190234a95?s=420&amp;d=https://a248.e.akamai.net/assets.github.com%2Fimages%2Fgravatars%2Fgravatar-user-420.png"/>
-    <meta property="og:site_name" content="GitHub"/>
-    <meta property="og:description" content="Gen2_Platforms_old - Generatioin 2 Platform Code Base"/>
-    <meta property="twitter:card" content="summary"/>
-    <meta property="twitter:site" content="@GitHub">
-    <meta property="twitter:title" content="crrlab368/Gen2_Platforms_old"/>
-    <meta name="description" content="Gen2_Platforms_old - Generatioin 2 Platform Code Base" />
-    <meta content="954816" name="octolytics-dimension-user_id" /><meta content="2144474" name="octolytics-dimension-repository_id" />
-  <link href="https://github.com/crrlab368/Gen2_Platforms_old/commits/master.atom" rel="alternate" title="Recent Commits to Gen2_Platforms_old:master" type="application/atom+xml" />
-  </head>
-  <body class="logged_in page-blob linux vis-public env-production  ">
-    <div id="wrapper">
-      <div class="header header-logged-in true">
-  <div class="container clearfix">
-    <a class="header-logo-invertocat" href="https://github.com/">
-  <span class="mega-octicon octicon-mark-github"></span>
-</a>
-    <div class="divider-vertical"></div>
-      <a href="/notifications" class="notification-indicator tooltipped downwards" title="You have no unread notifications">
-    <span class="mail-status all-read"></span>
-  </a>
-  <div class="divider-vertical"></div>
-      <div class="command-bar js-command-bar  in-repository">
-          <form accept-charset="UTF-8" action="/search" class="command-bar-form" id="top_search_form" method="get">
-  <a href="/search/advanced" class="advanced-search-icon tooltipped downwards command-bar-search" id="advanced_search" title="Advanced search"><span class="octicon octicon-gear "></span></a>
-  <input type="text" data-hotkey="/ s" name="q" id="js-command-bar-field" placeholder="Search or type a command" tabindex="1" autocapitalize="off"
-    data-username="crrlab368"
-      data-repo="crrlab368/Gen2_Platforms_old"
-      data-branch="master"
-      data-sha="d65dfc5c06acd8a403f58cbeef8a5fb3f69dd4dc"
-  >
-    <input type="hidden" name="nwo" value="crrlab368/Gen2_Platforms_old" />
-    <div class="select-menu js-menu-container js-select-menu search-context-select-menu">
-      <span class="minibutton select-menu-button js-menu-target">
-        <span class="js-select-button">This repository</span>
-      </span>
-      <div class="select-menu-modal-holder js-menu-content js-navigation-container">
-        <div class="select-menu-modal">
-          <div class="select-menu-item js-navigation-item selected">
-            <span class="select-menu-item-icon octicon octicon-check"></span>
-            <input type="radio" class="js-search-this-repository" name="search_target" value="repository" checked="checked" />
-            <div class="select-menu-item-text js-select-button-text">This repository</div>
-          </div> <!-- /.select-menu-item -->
-          <div class="select-menu-item js-navigation-item">
-            <span class="select-menu-item-icon octicon octicon-check"></span>
-            <input type="radio" name="search_target" value="global" />
-            <div class="select-menu-item-text js-select-button-text">All repositories</div>
-          </div> <!-- /.select-menu-item -->
-        </div>
-      </div>
-    </div>
-  <span class="octicon help tooltipped downwards" title="Show command bar help">
-    <span class="octicon octicon-question"></span>
-  </span>
-  <input type="hidden" name="ref" value="cmdform">
-  <div class="divider-vertical"></div>
-</form>
-        <ul class="top-nav">
-            <li class="explore"><a href="https://github.com/explore">Explore</a></li>
-            <li><a href="https://gist.github.com">Gist</a></li>
-            <li><a href="/blog">Blog</a></li>
-          <li><a href="http://help.github.com">Help</a></li>
-        </ul>
-      </div>
-    <ul id="user-links">
-      <li>
-        <a href="https://github.com/crrlab368" class="name">
-          <img height="20" src="https://secure.gravatar.com/avatar/9f67947d0c852e39e3bd1cf190234a95?s=140&amp;d=https://a248.e.akamai.net/assets.github.com%2Fimages%2Fgravatars%2Fgravatar-user-420.png" width="20" /> crrlab368
-        </a>
-      </li>
-        <li>
-          <a href="/new" id="new_repo" class="tooltipped downwards" title="Create a new repo">
-            <span class="octicon octicon-repo-create"></span>
-          </a>
-        </li>
-        <li>
-          <a href="/settings/profile" id="account_settings"
-            class="tooltipped downwards"
-            title="Account settings ">
-            <span class="octicon octicon-tools"></span>
-          </a>
-        </li>
-        <li>
-          <a class="tooltipped downwards" href="/logout" data-method="post" id="logout" title="Sign out">
-            <span class="octicon octicon-log-out"></span>
-          </a>
-        </li>
-    </ul>
-<div class="js-new-dropdown-contents hidden">
-  <ul class="dropdown-menu">
-    <li>
-      <a href="/new"><span class="octicon octicon-repo-create"></span> New repository</a>
-    </li>
-    <li>
-        <a href="https://github.com/crrlab368/Gen2_Platforms_old/issues/new"><span class="octicon octicon-issue-opened"></span> New issue</a>
-    </li>
-    <li>
-    </li>
-    <li>
-      <a href="/organizations/new"><span class="octicon octicon-list-unordered"></span> New organization</a>
-    </li>
-  </ul>
-</div>
-  </div>
-</div>
-            <div class="site hfeed" itemscope itemtype="http://schema.org/WebPage">
-      <div class="hentry">
-        <div class="pagehead repohead instapaper_ignore readability-menu ">
-          <div class="container">
-            <div class="title-actions-bar">
-<ul class="pagehead-actions">
-    <li class="nspr">
-      <a href="/crrlab368/Gen2_Platforms_old/pull/new/master" class="button minibutton btn-pull-request" icon_class="octicon-git-pull-request"><span class="octicon octicon-git-pull-request"></span>Pull Request</a>
-    </li>
-    <li class="subscription">
-      <form accept-charset="UTF-8" action="/notifications/subscribe" data-autosubmit="true" data-remote="true" method="post"><div style="margin:0;padding:0;display:inline"><input name="authenticity_token" type="hidden" value="vWZ31DoCO0bdiK1SaFbgMAphXvwWP/Ea7z/IJlIrUBA=" /></div>  <input id="repository_id" name="repository_id" type="hidden" value="2144474" />
-    <div class="select-menu js-menu-container js-select-menu">
-      <span class="minibutton select-menu-button js-menu-target">
-        <span class="js-select-button">
-          <span class="octicon octicon-eye-unwatch"></span>
-          Unwatch
-        </span>
-      </span>
-      <div class="select-menu-modal-holder js-menu-content">
-        <div class="select-menu-modal">
-          <div class="select-menu-header">
-            <span class="select-menu-title">Notification status</span>
-            <span class="octicon octicon-remove-close js-menu-close"></span>
-          </div> <!-- /.select-menu-header -->
-          <div class="select-menu-list js-navigation-container">
-            <div class="select-menu-item js-navigation-item ">
-              <span class="select-menu-item-icon octicon octicon-check"></span>
-              <div class="select-menu-item-text">
-                <input id="do_included" name="do" type="radio" value="included" />
-                <h4>Not watching</h4>
-                <span class="description">You only receive notifications for discussions in which you participate or are @mentioned.</span>
-                <span class="js-select-button-text hidden-select-button-text">
-                  <span class="octicon octicon-eye-watch"></span>
-                  Watch
-                </span>
-              </div>
-            </div> <!-- /.select-menu-item -->
-            <div class="select-menu-item js-navigation-item selected">
-              <span class="select-menu-item-icon octicon octicon octicon-check"></span>
-              <div class="select-menu-item-text">
-                <input checked="checked" id="do_subscribed" name="do" type="radio" value="subscribed" />
-                <h4>Watching</h4>
-                <span class="description">You receive notifications for all discussions in this repository.</span>
-                <span class="js-select-button-text hidden-select-button-text">
-                  <span class="octicon octicon-eye-unwatch"></span>
-                  Unwatch
-                </span>
-              </div>
-            </div> <!-- /.select-menu-item -->
-            <div class="select-menu-item js-navigation-item ">
-              <span class="select-menu-item-icon octicon octicon-check"></span>
-              <div class="select-menu-item-text">
-                <input id="do_ignore" name="do" type="radio" value="ignore" />
-                <h4>Ignoring</h4>
-                <span class="description">You do not receive any notifications for discussions in this repository.</span>
-                <span class="js-select-button-text hidden-select-button-text">
-                  <span class="octicon octicon-mute"></span>
-                  Stop ignoring
-                </span>
-              </div>
-            </div> <!-- /.select-menu-item -->
-          </div> <!-- /.select-menu-list -->
-        </div> <!-- /.select-menu-modal -->
-      </div> <!-- /.select-menu-modal-holder -->
-    </div> <!-- /.select-menu -->
-</form>
-    </li>
-    <li class="js-toggler-container js-social-container starring-container on">
-      <a href="/crrlab368/Gen2_Platforms_old/unstar" class="minibutton js-toggler-target star-button starred upwards" title="Unstar this repo" data-remote="true" data-method="post" rel="nofollow">
-        <span class="octicon octicon-star-delete"></span>
-        <span class="text">Unstar</span>
-      </a>
-      <a href="/crrlab368/Gen2_Platforms_old/star" class="minibutton js-toggler-target star-button unstarred upwards" title="Star this repo" data-remote="true" data-method="post" rel="nofollow">
-        <span class="octicon octicon-star"></span>
-        <span class="text">Star</span>
-      </a>
-      <a class="social-count js-social-count" href="/crrlab368/Gen2_Platforms_old/stargazers">2</a>
-    </li>
-        <li>
-          <a href="/crrlab368/Gen2_Platforms_old/fork" class="minibutton js-toggler-target fork-button lighter upwards" title="Fork this repo" rel="nofollow" data-method="post">
-            <span class="octicon octicon-git-branch-create"></span>
-            <span class="text">Fork</span>
-          </a>
-          <a href="/crrlab368/Gen2_Platforms_old/network" class="social-count">0</a>
-        </li>
-</ul>
-              <h1 itemscope itemtype="http://data-vocabulary.org/Breadcrumb" class="entry-title public">
-                <span class="repo-label"><span>public</span></span>
-                <span class="mega-octicon octicon-repo"></span>
-                <span class="author vcard">
-                  <a href="/crrlab368" class="url fn" itemprop="url" rel="author">
-                  <span itemprop="title">crrlab368</span>
-                  </a></span> /
-                <strong><a href="/crrlab368/Gen2_Platforms_old" class="js-current-repository">Gen2_Platforms_old</a></strong>
-              </h1>
-            </div>
-  <ul class="tabs">
-    <li class="pulse-nav"><a href="/crrlab368/Gen2_Platforms_old/pulse" class="js-selected-navigation-item " data-selected-links="pulse /crrlab368/Gen2_Platforms_old/pulse" rel="nofollow"><span class="octicon octicon-pulse"></span></a></li>
-    <li><a href="/crrlab368/Gen2_Platforms_old" class="js-selected-navigation-item selected" data-selected-links="repo_source repo_downloads repo_commits repo_tags repo_branches /crrlab368/Gen2_Platforms_old">Code</a></li>
-    <li><a href="/crrlab368/Gen2_Platforms_old/network" class="js-selected-navigation-item " data-selected-links="repo_network /crrlab368/Gen2_Platforms_old/network">Network</a></li>
-    <li><a href="/crrlab368/Gen2_Platforms_old/pulls" class="js-selected-navigation-item " data-selected-links="repo_pulls /crrlab368/Gen2_Platforms_old/pulls">Pull Requests <span class='counter'>0</span></a></li>
-      <li><a href="/crrlab368/Gen2_Platforms_old/issues" class="js-selected-navigation-item " data-selected-links="repo_issues /crrlab368/Gen2_Platforms_old/issues">Issues <span class='counter'>0</span></a></li>
-      <li><a href="/crrlab368/Gen2_Platforms_old/wiki" class="js-selected-navigation-item " data-selected-links="repo_wiki /crrlab368/Gen2_Platforms_old/wiki">Wiki</a></li>
-    <li><a href="/crrlab368/Gen2_Platforms_old/graphs" class="js-selected-navigation-item " data-selected-links="repo_graphs repo_contributors /crrlab368/Gen2_Platforms_old/graphs">Graphs</a></li>
-      <li>
-        <a href="/crrlab368/Gen2_Platforms_old/settings">Settings</a>
-      </li>
-  </ul>
-<div class="tabnav">
-  <span class="tabnav-right">
-    <ul class="tabnav-tabs">
-          <li><a href="/crrlab368/Gen2_Platforms_old/tags" class="js-selected-navigation-item tabnav-tab" data-selected-links="repo_tags /crrlab368/Gen2_Platforms_old/tags">Tags <span class="counter blank">0</span></a></li>
-    </ul>
-  </span>
-  <div class="tabnav-widget scope">
-    <div class="select-menu js-menu-container js-select-menu js-branch-menu">
-      <a class="minibutton select-menu-button js-menu-target" data-hotkey="w" data-ref="master">
-        <span class="octicon octicon-branch"></span>
-        <i>branch:</i>
-        <span class="js-select-button">master</span>
-      </a>
-      <div class="select-menu-modal-holder js-menu-content js-navigation-container">
-        <div class="select-menu-modal">
-          <div class="select-menu-header">
-            <span class="select-menu-title">Switch branches/tags</span>
-            <span class="octicon octicon-remove-close js-menu-close"></span>
-          </div> <!-- /.select-menu-header -->
-          <div class="select-menu-filters">
-            <div class="select-menu-text-filter">
-              <input type="text" id="commitish-filter-field" class="js-filterable-field js-navigation-enable" placeholder="Find or create a branch…">
-            </div>
-            <div class="select-menu-tabs">
-              <ul>
-                <li class="select-menu-tab">
-                  <a href="#" data-tab-filter="branches" class="js-select-menu-tab">Branches</a>
-                </li>
-                <li class="select-menu-tab">
-                  <a href="#" data-tab-filter="tags" class="js-select-menu-tab">Tags</a>
-                </li>
-              </ul>
-            </div><!-- /.select-menu-tabs -->
-          </div><!-- /.select-menu-filters -->
-          <div class="select-menu-list select-menu-tab-bucket js-select-menu-tab-bucket css-truncate" data-tab-filter="branches">
-            <div data-filterable-for="commitish-filter-field" data-filterable-type="substring">
-                <div class="select-menu-item js-navigation-item selected">
-                  <span class="select-menu-item-icon octicon octicon-check"></span>
-                  <a href="/crrlab368/Gen2_Platforms_old/blob/master/gen2_common/gen2_description/urdf/gen2.xacro" class="js-navigation-open select-menu-item-text js-select-button-text css-truncate-target" data-name="master" rel="nofollow" title="master">master</a>
-                </div> <!-- /.select-menu-item -->
-            </div>
-              <form accept-charset="UTF-8" action="/crrlab368/Gen2_Platforms_old/branches" class="js-create-branch select-menu-item select-menu-new-item-form js-navigation-item js-new-item-form" method="post"><div style="margin:0;padding:0;display:inline"><input name="authenticity_token" type="hidden" value="vWZ31DoCO0bdiK1SaFbgMAphXvwWP/Ea7z/IJlIrUBA=" /></div>
-                <span class="octicon octicon-git-branch-create select-menu-item-icon"></span>
-                <div class="select-menu-item-text">
-                  <h4>Create branch: <span class="js-new-item-name"></span></h4>
-                  <span class="description">from ‘master’</span>
-                </div>
-                <input type="hidden" name="name" id="name" class="js-new-item-value">
-                <input type="hidden" name="branch" id="branch" value="master" />
-                <input type="hidden" name="path" id="branch" value="gen2_common/gen2_description/urdf/gen2.xacro" />
-              </form> <!-- /.select-menu-item -->
-          </div> <!-- /.select-menu-list -->
-          <div class="select-menu-list select-menu-tab-bucket js-select-menu-tab-bucket css-truncate" data-tab-filter="tags">
-            <div data-filterable-for="commitish-filter-field" data-filterable-type="substring">
-            </div>
-            <div class="select-menu-no-results">Nothing to show</div>
-          </div> <!-- /.select-menu-list -->
-        </div> <!-- /.select-menu-modal -->
-      </div> <!-- /.select-menu-modal-holder -->
-    </div> <!-- /.select-menu -->
-  </div> <!-- /.scope -->
-  <ul class="tabnav-tabs">
-    <li><a href="/crrlab368/Gen2_Platforms_old" class="selected js-selected-navigation-item tabnav-tab" data-selected-links="repo_source /crrlab368/Gen2_Platforms_old">Files</a></li>
-    <li><a href="/crrlab368/Gen2_Platforms_old/commits/master" class="js-selected-navigation-item tabnav-tab" data-selected-links="repo_commits /crrlab368/Gen2_Platforms_old/commits/master">Commits</a></li>
-    <li><a href="/crrlab368/Gen2_Platforms_old/branches" class="js-selected-navigation-item tabnav-tab" data-selected-links="repo_branches /crrlab368/Gen2_Platforms_old/branches" rel="nofollow">Branches <span class="counter ">1</span></a></li>
-  </ul>
-</div>
-          </div>
-        </div><!-- /.repohead -->
-        <div id="js-repo-pjax-container" class="container context-loader-container" data-pjax-container>
-<!-- blob contrib key: blob_contributors:v21:ad254e30f03f2a651986d60cd6f35e1e -->
-<!-- blob contrib frag key: views10/v8/blob_contributors:v21:ad254e30f03f2a651986d60cd6f35e1e -->
-<div id="slider">
-    <div class="frame-meta">
-      <p title="This is a placeholder element" class="js-history-link-replace hidden"></p>
-        <div class="breadcrumb">
-          <span class='bold'><span itemscope="" itemtype="http://data-vocabulary.org/Breadcrumb"><a href="/crrlab368/Gen2_Platforms_old" class="js-slide-to" data-branch="master" data-direction="back" itemscope="url"><span itemprop="title">Gen2_Platforms_old</span></a></span></span><span class="separator"> / </span><span itemscope="" itemtype="http://data-vocabulary.org/Breadcrumb"><a href="/crrlab368/Gen2_Platforms_old/tree/master/gen2_common" class="js-slide-to" data-branch="master" data-direction="back" itemscope="url"><span itemprop="title">gen2_common</span></a></span><span class="separator"> / </span><span itemscope="" itemtype="http://data-vocabulary.org/Breadcrumb"><a href="/crrlab368/Gen2_Platforms_old/tree/master/gen2_common/gen2_description" class="js-slide-to" data-branch="master" data-direction="back" itemscope="url"><span itemprop="title">gen2_description</span></a></span><span class="separator"> / </span><span itemscope="" itemtype="http://data-vocabulary.org/Breadcrumb"><a href="/crrlab368/Gen2_Platforms_old/tree/master/gen2_common/gen2_description/urdf" class="js-slide-to" data-branch="master" data-direction="back" itemscope="url"><span itemprop="title">urdf</span></a></span><span class="separator"> / </span><strong class="final-path">gen2.xacro</strong> <span class="js-zeroclipboard zeroclipboard-button" data-clipboard-text="gen2_common/gen2_description/urdf/gen2.xacro" data-copied-hint="copied!" title="copy to clipboard"><span class="octicon octicon-clippy"></span></span>
-        </div>
-      <a href="/crrlab368/Gen2_Platforms_old/find/master" class="js-slide-to" data-hotkey="t" style="display:none">Show File Finder</a>
-  <div class="commit file-history-tease">
-    <img class="main-avatar" height="24" src="https://secure.gravatar.com/avatar/9f67947d0c852e39e3bd1cf190234a95?s=140&amp;d=https://a248.e.akamai.net/assets.github.com%2Fimages%2Fgravatars%2Fgravatar-user-420.png" width="24" />
-    <span class="author"><a href="/crrlab368" rel="author">crrlab368</a></span>
-    <time class="js-relative-date" datetime="2011-09-01T08:46:48-07:00" title="2011-09-01 08:46:48">September 01, 2011</time>
-    <div class="commit-title">
-        <a href="/crrlab368/Gen2_Platforms_old/commit/c117a61a6d6666a4fed65707c96177add19b7aff" class="message">Fixed error in urdf</a>
-    </div>
-    <div class="participation">
-      <p class="quickstat"><a href="#blob_contributors_box" rel="facebox"><strong>1</strong> contributor</a></p>
-    </div>
-    <div id="blob_contributors_box" style="display:none">
-      <h2>Users on GitHub who have contributed to this file</h2>
-      <ul class="facebox-user-list">
-        <li>
-          <img height="24" src="https://secure.gravatar.com/avatar/9f67947d0c852e39e3bd1cf190234a95?s=140&amp;d=https://a248.e.akamai.net/assets.github.com%2Fimages%2Fgravatars%2Fgravatar-user-420.png" width="24" />
-          <a href="/crrlab368">crrlab368</a>
-        </li>
-      </ul>
-    </div>
-  </div>
-    </div><!-- ./.frame-meta -->
-    <div class="frames">
-      <div class="frame" data-permalink-url="/crrlab368/Gen2_Platforms_old/blob/5cf94742cfdbf212b6ec9cc24dc8148d8ee83f12/gen2_common/gen2_description/urdf/gen2.xacro" data-title="Gen2_Platforms_old/gen2_common/gen2_description/urdf/gen2.xacro at master · crrlab368/Gen2_Platforms_old · GitHub" data-type="blob">
-        <div id="files" class="bubble">
-          <div class="file">
-            <div class="meta">
-              <div class="info">
-                <span class="icon"><b class="octicon octicon-file-text"></b></span>
-                <span class="mode" title="File Mode">file</span>
-                  <span>676 lines (550 sloc)</span>
-                <span>15.733 kb</span>
-              </div>
-              <div class="actions">
-                <div class="button-group">
-                        <a class="minibutton"
-                           href="/crrlab368/Gen2_Platforms_old/edit/master/gen2_common/gen2_description/urdf/gen2.xacro"
-                           data-method="post" rel="nofollow" data-hotkey="e">Edit</a>
-                  <a href="/crrlab368/Gen2_Platforms_old/raw/master/gen2_common/gen2_description/urdf/gen2.xacro" class="button minibutton " id="raw-url">Raw</a>
-                    <a href="/crrlab368/Gen2_Platforms_old/blame/master/gen2_common/gen2_description/urdf/gen2.xacro" class="button minibutton ">Blame</a>
-                  <a href="/crrlab368/Gen2_Platforms_old/commits/master/gen2_common/gen2_description/urdf/gen2.xacro" class="button minibutton " rel="nofollow">History</a>
-                </div><!-- /.button-group -->
-              </div><!-- /.actions -->
-            </div>
-                <div class="blob-wrapper data type-text js-blob-data">
-      <table class="file-code file-diff">
-        <tr class="file-code-line">
-          <td class="blob-line-nums">
-            <span id="L1" rel="#L1">1</span>
-<span id="L2" rel="#L2">2</span>
-<span id="L3" rel="#L3">3</span>
-<span id="L4" rel="#L4">4</span>
-<span id="L5" rel="#L5">5</span>
-<span id="L6" rel="#L6">6</span>
-<span id="L7" rel="#L7">7</span>
-<span id="L8" rel="#L8">8</span>
-<span id="L9" rel="#L9">9</span>
-<span id="L10" rel="#L10">10</span>
-<span id="L11" rel="#L11">11</span>
-<span id="L12" rel="#L12">12</span>
-<span id="L13" rel="#L13">13</span>
-<span id="L14" rel="#L14">14</span>
-<span id="L15" rel="#L15">15</span>
-<span id="L16" rel="#L16">16</span>
-<span id="L17" rel="#L17">17</span>
-<span id="L18" rel="#L18">18</span>
-<span id="L19" rel="#L19">19</span>
-<span id="L20" rel="#L20">20</span>
-<span id="L21" rel="#L21">21</span>
-<span id="L22" rel="#L22">22</span>
-<span id="L23" rel="#L23">23</span>
-<span id="L24" rel="#L24">24</span>
-<span id="L25" rel="#L25">25</span>
-<span id="L26" rel="#L26">26</span>
-<span id="L27" rel="#L27">27</span>
-<span id="L28" rel="#L28">28</span>
-<span id="L29" rel="#L29">29</span>
-<span id="L30" rel="#L30">30</span>
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